File: hw/lab7811_project/lab7811_project.kicad_sch (KiCad schematic)
At the start: 38 parts, among them J1 Battery, J2 JTAG, J3 Conn_01x08_Pin, SW1 Start, SW2 Reset, SW4 Reset, U1 MPU-6050, U2 TM4C123GH6PMIR, U3 FT232RL-REEL, U4 LP2950-33LPRE3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

Commit message: new footprints
Parts:
- U1: footprint Sensor_Motion:InvenSense_QFN-24_4x4mm_P0.5mm -> gyroLibrary:PinHeader_1x08_P2.54mm_Vertical
