File: hw/lab7811_project/lab7811_project.kicad_sch (KiCad schematic)
At the start: 41 parts, among them J1 Conn_01x06, J2 JTAG, J3 Conn_01x08_Pin, SW1 Start, SW3 Up, SW4 Reset, SW5 Down, SW6 Left, SW7 Right, U1 MPU-6050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

Commit message: finished schematic and pcb for TA review
Parts:
- removed J1: Conn_01x06, symbol Connector_Generic:Conn_01x06
- added J1: Conn_01x05, Connector_PinHeader_2.54mm:PinHeader_1x05_P2.54mm_Vertical, symbol Connector_Generic:Conn_01x05
Connections:
- net +3.3V is gone; now on net +3V3: R3.1, R4.1, R7.1, R8.1, R9.1, U1.13 (VDD)
- net GND: now also J1.5 (GND)
- net PB0: now also J1.4 (IO)
- net PB4: now also J3.3 (Pin_3)
- net PB5: now also J3.4 (Pin_4)
- net PD4: now also J1.2 (D-)
- net PD5: now also J1.3 (D+)
- net PE4: no longer J3.3 (Pin_3)
- net PE5: no longer J3.4 (Pin_4)
- net at C1.1, U4.3 (INPUT): now also J1.1 (VBUS)
- no-connect marks 18 -> 16
Other:
- moved on the sheet: U1
