File: hw/lab7811_project/_autosave-lab7811_project.kicad_sch (KiCad schematic)
At the start: 41 parts, among them J1 Conn_01x06, J2 JTAG, J3 Conn_01x08_Pin, SW1 Start, SW3 Up, SW4 Reset, SW5 Down, SW6 Left, SW7 Right, U1 MPU-6050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

Commit message: updated the schematic
Parts:
- J1: footprint (none) -> Connector_PinHeader_2.54mm:PinHeader_1x06_P2.54mm_Vertical
Changed lines of the file:
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@@
       (effects (font (size 1.27 1.27)) (justify left))
     )
-    (property "Footprint" "" (at 35.56 71.12 0)
+    (property "Footprint" "Connector_PinHeader_2.54mm:PinHeader_1x06_P2.54mm_Vertical" (at 35.56 71.12 0)
       (effects (font (size 1.27 1.27)) hide)
     )
