File: hw/lab7811_project/lab7811_project.kicad_pcb (KiCad board)
At the start: 2 copper layers, 37 parts, among them J1 Battery, J2 JTAG, J3 Conn_01x08_Pin, SW1 Start, SW2 Reset, SW4 Reset, U1 MPU-6050, U2 TM4C123GH6PMIR, U4 LP2950-33LPRE3, U5 Adafruit ST7735R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

Commit message: new footprints
Parts:
- moved U1 68.8 mm to (115.6, 52.1)

Commit message: updated the schematic
Parts:
- removed R2: 10k, ECE445L:R_Axial_DIN0204_L3.6mm_D1.6mm_P7.62mm_Horizontal
- removed SW2: Reset, ECE445L:SW_PUSH_6mm
- removed TP1: GND, ECE445L:Testpoint_1x02_P2.54mm
- removed TP2: +3.7V, ECE445L:Testpoint_1x02_P2.54mm
- added R4: 10k, ECE445L:R_Axial_DIN0204_L3.6mm_D1.6mm_P7.62mm_Horizontal, F.Cu at (112.5, 73.7)
- added R7: 10k, ECE445L:R_Axial_DIN0204_L3.6mm_D1.6mm_P7.62mm_Horizontal, F.Cu at (128.8, 99.1)
- added R8: 10k, ECE445L:R_Axial_DIN0204_L3.6mm_D1.6mm_P7.62mm_Horizontal, F.Cu at (112.5, 99.1)
- added R9: 10k, ECE445L:R_Axial_DIN0204_L3.6mm_D1.6mm_P7.62mm_Horizontal, F.Cu at (128.8, 73.7)
- added SW3: Up, ECE445L:SW_PUSH_6mm, F.Cu at (116.1, 76.5)
- added SW5: Down, ECE445L:SW_PUSH_6mm, F.Cu at (116.1, 91.7)
- added SW6: Left, ECE445L:SW_PUSH_6mm, F.Cu at (106.0, 84.1)
- added SW7: Right, ECE445L:SW_PUSH_6mm, F.Cu at (125.6, 84.2)
- C10, C11, C12, C13, C3, C4, C5, C6, C7, C8, C9, U1, Y1: moved to B.Cu
- J1: value Battery -> Conn_01x06; footprint ECE445L:PinHeader_1x02_P2.54mm_Vertical -> Connector_PinHeader_2.54mm:PinHeader_1x06_P2.54mm_Vertical; moved to B.Cu
- moved SW4 108.4 mm to (179.6, 91.7)
- moved U5 103.5 mm to (153.0, 78.7)
- moved SW1 102.5 mm to (178.9, 59.0)
- moved C12 99.6 mm to (170.2, 81.3)
- moved C11 99.6 mm to (170.2, 76.2)
- moved R3 97.3 mm to (175.3, 68.6), turned to 90 degrees
- moved D1 93.8 mm to (124.5, 58.4)
- moved R6 93.7 mm to (172.7, 101.6)
- moved R5 93.5 mm to (172.7, 96.5), turned to 90 degrees
- moved C10 91.6 mm to (157.5, 91.4), turned to -90 degrees
- moved C5 91.4 mm to (148.0, 91.4), turned to -90 degrees
- moved C8 90.6 mm to (152.4, 91.4), turned to -90 degrees
- moved C9 86.9 mm to (157.5, 66.0), turned to 90 degrees
- moved C3 86.7 mm to (142.2, 81.9), turned to 180 degrees
- moved J2 84.3 mm to (152.4, 55.9), turned to 90 degrees
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Connections:
- C1 pad 1: /+3_7V -> Net-(J1-VCC)
- J1 pad 1: GND -> Net-(J1-VCC)
- J1 pad 2: /+3_7V -> GND
- J3 pad 1: PA5 -> PE2
- J3 pad 2: PA4 -> PE3
- J3 pad 3: PA2 -> PE4
- J3 pad 4: PD3 -> PE5
- J3 pad 5: PD1 -> PD2
- J3 pad 6: PD0 -> PD1
- J3 pad 7: PE1 -> PD0
- J3 pad 8: PE0 -> unconnected-(J3-Pin_8-Pad8)
- R3 pad 2: PE2 -> PD2
- SW1 pad 1: PE2 -> PD2
- U4 pad 3: /+3_7V -> Net-(J1-VCC)
Routing:
- net GND: track 0.00 -> 1.12 mm

Commit message: finished schematic and pcb for TA review
Parts:
- removed H4: ~, ECE445L:MountingHole_4_40
- J1: value Conn_01x06 -> Conn_01x05; footprint Connector_PinHeader_2.54mm:PinHeader_1x06_P2.54mm_Vertical -> Connector_PinHeader_2.54mm:PinHeader_1x05_P2.54mm_Vertical; moved to F.Cu
- moved H3 52.8 mm to (165.1, 91.4)
- moved H2 51.1 mm to (139.7, 96.5)
- moved H1 27.7 mm to (132.1, 66.0)
- moved TP3 22.9 mm to (106.7, 67.7), turned to 0 degrees
- moved R1 22.6 mm to (118.1, 71.1), turned to 0 degrees
- moved C2 20.5 mm to (106.7, 73.7)
- moved J2 20.5 mm to (172.7, 53.3)
- moved U4 14.4 mm to (106.7, 63.5), turned to 90 degrees
- moved J1 10.5 mm to (116.8, 55.9), turned to 90 degrees
- moved D1 5.68 mm to (121.9, 63.5)
- moved C1 3.59 mm to (114.3, 63.5), turned to -90 degrees
- moved R3 2.84 mm to (172.7, 69.8)
- moved SW4 2.54 mm to (177.1, 91.7)
- moved SW1 1.83 mm to (177.1, 59.0)
Connections:
- J1 pad 2: GND -> PD4
- J1 pad 3: PE4 -> PD5
- J1 pad 4: PE5 -> PB0
- J1 pad 5: unconnected-(J1-RTS-Pad5) -> GND
- J3 pad 3: PE4 -> PB4
- J3 pad 4: PE5 -> PB5
- R3 pad 1: +3.3V -> +3V3
- R4 pad 1: +3.3V -> +3V3
- R7 pad 1: +3.3V -> +3V3
- R8 pad 1: +3.3V -> +3V3
- R9 pad 1: +3.3V -> +3V3
- U1 pad 13: +3.3V -> +3V3
Routing:
- net GND: track 1.12 -> 368.5 mm
- net +3V3: track 0.00 -> 308.6 mm, vias 0 -> 5
- net PB4: track 0.00 -> 174.5 mm
- net PD0: track 0.00 -> 116.8 mm, vias 0 -> 2
- net PE3: track 0.00 -> 112.1 mm
- net PD1: track 0.00 -> 111.8 mm, vias 0 -> 2
- net PB5: track 0.00 -> 106.0 mm, vias 0 -> 2
- net PD2: track 0.00 -> 97.7 mm, vias 0 -> 2
- net PE2: track 0.00 -> 66.5 mm
- net PD4: track 0.00 -> 65.7 mm, vias 0 -> 2
- net PD5: track 0.00 -> 64.4 mm, vias 0 -> 2
- net PB0: track 0.00 -> 60.0 mm, vias 0 -> 2
- net /LDO: track 0.00 -> 42.7 mm, vias 0 -> 2
- net /Reset: track 0.00 -> 41.5 mm
- net PD7: track 0.00 -> 35.9 mm
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Other:
- board outline added: 86.4 x 61 mm
